Commit message: se agrega todo el brazo

File: src/piper_description/urdf/piper_description.urdf (robot description, URDF)
Before this commit: robot piper, 10 links, 9 joints
Joints:
- joint joint7: limit lower=0 upper=0.035 effort=10 velocity=1 -> lower=0 upper=0.1 effort=10 velocity=1
- joint joint8: limit lower=-0.035 upper=0 effort=10 velocity=1 -> lower=-0.1 upper=0 effort=10 velocity=1
